File: PCIexpress_x16_half/PCIexpress_x16_half.kicad_pcb (KiCad board)
At the start: 4 copper layers, 312 x 111.2 mm, 66 parts, among them J1 PCIexpress_bracket, J2 PCIexpress_x16

Commit message: half x16
Other:
- board size 312 x 111.2 mm -> 167.7 x 111.2 mm
Changed lines of the file:
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@@
   (general
     (thickness 1.6)
-    (drawings 58)
+    (drawings 51)
     (tracks 425)
     (zones 0)
@@
     )
   )
-  (gr_circle (center 371.395 87.995) (end 372.995 87.995) (layer Edge.Cuts) (width 0.15))
-  (gr_circle (center 371.395 177.525) (end 372.995 177.525) (layer Edge.Cuts) (width 0.15))
+  (gr_line (start 232.1277 181.375) (end 205.525 181.375) (layer Edge.Cuts) (width 0.15))
+  (gr_line (start 232.125 82.975) (end 232.1277 181.375) (layer Edge.Cuts) (width 0.15))
+  (gr_line (start 64.475 82.975) (end 232.125 82.975) (layer Edge.Cuts) (width 0.15))
   (gr_line (start 69.555 104.425) (end 69.555 180.375) (layer Dwgs.User) (width 0.15))
   (gr_line (start 109.475 180.375) (end 109.475 193.625) (layer Dwgs.User) (width 0.15))
@@
   (gr_line (start 201.625 85.975) (end 201.625 83.975) (layer Dwgs.User) (width 0.15))
   (gr_line (start 366.275 85.975) (end 201.625 85.975) (layer Dwgs.User) (width 0.15))
-  (gr_line (start 366.275 94.425) (end 366.275 85.975) (layer Dwgs.User) (width 0.15))
-  (gr_line (start 371.395 94.425) (end 366.275 94.425) (layer Dwgs.User) (width 0.15))
-  (gr_line (start 371.395 171.225) (end 371.395 94.425) (layer Dwgs.User) (width 0.15))
-  (gr_line (start 366.275 171.225) (end 371.395 171.225) (layer Dwgs.User) (width 0.15))
-  (gr_line (start 366.275 180.375) (end 366.275 171.225) (layer Dwgs.User) (width 0.15))
   (gr_line (start 219.925 180.375) (end 366.275 180.375) (layer Dwgs.User) (width 0.15))
   (gr_line (start 219.925 178.025) (end 219.925 180.375) (layer Dwgs.User) (width 0.15))
@@
   (gr_line (start 64.475 189.625) (end 79.475 189.625) (layer Edge.Cuts) (width 0.15))
   (gr_line (start 64.475 82.975) (end 64.475 189.625) (layer Edge.Cuts) (width 0.15))
-  (gr_line (start 376.475 82.975) (end 64.475 82.975) (layer Edge.Cuts) (width 0.15))
-  (gr_line (start 376.4777 181.375) (end 376.475 82.975) (layer Edge.Cuts) (width 0.15))
-  (gr_line (start 205.525 181.375) (end 376.4777 181.375) (layer Edge.Cuts) (width 0.15))
   (gr_line (start 203.775 184.425) (end 203.775 183.125) (layer Edge.Cuts) (width 0.15))
   (gr_line (start 209.225 186.175) (end 205.525 186.175) (layer Edge.Cuts) (width 0.15))
@@
     (polygon
       (pts
-        (xy 193.775 186.175) (xy 193.775 180.375) (xy 366.275 180.375) (xy 366.275 171.225) (xy 371.395 171.225)
-        (xy 371.395 94.425) (xy 366.275 94.425) (xy 366.275 85.975) (xy 201.625 85.975) (xy 201.625 83.975)
-        (xy 77.175 83.975) (xy 77.175 104.425) (xy 64.475 104.425) (xy 64.475 82.975) (xy 376.475 82.975)
-        (xy 376.4777 181.375) (xy 205.525 181.375) (xy 205.525 186.175) (xy 196.525 186.175)
-      )
-    )
-  )
-  (zone (net 0) (net_name "") (layers F.Cu In1.Cu In2.Cu B.Cu) (hatch edge 0.508)
-    (connect_pads (clearance 0))
-    (min_thickness 0.254)
-    (keepout (tracks not_allowed) (vias not_allowed) (copperpour allowed))
-    (fill (arc_segments 32) (thermal_gap 0.508) (thermal_bridge_width 0.508))
-    (polygon
-      (pts
         (xy 64.475 180.375) (xy 109.475 180.375) (xy 109.475 183.2) (xy 105.825 183.2) (xy 105.825 186.125)
         (xy 97.825 186.125) (xy 97.825 181.375) (xy 79.475 181.375) (xy 79.475 189.625) (xy 64.475 189.625)
@@
     (polygon
       (pts
-        (xy 64.5 83) (xy 376.5 83) (xy 376.5 181.375) (xy 205.5 181.375) (xy 205.5 186.25)
+        (xy 64.5 83) (xy 232.125 83) (xy 232.125 181.375) (xy 205.5 181.375) (xy 205.5 186.25)
         (xy 193.75 186.25) (xy 193.75 188.625) (xy 109.375 188.625) (xy 109.375 183.25) (xy 105.875 183.25)
         (xy 105.875 186.125) (xy 97.75 186.125) (xy 97.75 181.375) (xy 79.5 181.375) (xy 79.5 189.625)
@@
     (polygon
       (pts
-        (xy 64.5 83) (xy 376.5 83) (xy 376.5 181.375) (xy 205.5 181.375) (xy 205.5 186.25)
+        (xy 64.5 83) (xy 232.125 83) (xy 232.125 181.375) (xy 205.5 181.375) (xy 205.5 186.25)
         (xy 193.75 186.25) (xy 193.75 188.625) (xy 109.375 188.625) (xy 109.375 183.25) (xy 105.875 183.25)
         (xy 105.875 186.125) (xy 97.75 186.125) (xy 97.75 181.375) (xy 79.5 181.375) (xy 79.5 189.625)
@@
     (polygon
       (pts
-        (xy 64.5 83) (xy 376.5 83) (xy 376.5 181.375) (xy 205.5 181.375) (xy 205.5 186.25)
+        (xy 64.5 83) (xy 232.125 83) (xy 232.125 181.375) (xy 205.5 181.375) (xy 205.5 186.25)
         (xy 193.75 186.25) (xy 193.75 188.625) (xy 109.375 188.625) (xy 109.375 183.25) (xy 105.875 183.25)
         (xy 105.875 186.125) (xy 97.75 186.125) (xy 97.75 181.375) (xy 79.5 181.375) (xy 79.5 189.625)
@@
     (polygon
       (pts
-        (xy 64.5 83) (xy 376.5 83) (xy 376.5 181.375) (xy 205.5 181.375) (xy 205.5 186.25)
+        (xy 64.5 83) (xy 232.125 83) (xy 232.125 181.375) (xy 205.5 181.375) (xy 205.5 186.25)
         (xy 193.75 186.25) (xy 193.75 188.625) (xy 109.375 188.625) (xy 109.375 183.25) (xy 105.875 183.25)
         (xy 105.875 186.125) (xy 97.75 186.125) (xy 97.75 181.375) (xy 79.5 181.375) (xy 79.5 189.625)
@@
       )
     )
+  )
+  (zone (net 0) (net_name "") (layers F.Cu In1.Cu In2.Cu B.Cu) (hatch edge 0.508)
+    (connect_pads (clearance 0.508))
+    (min_thickness 0.254)
+    (keepout (tracks not_allowed) (vias not_allowed) (copperpour allowed))
+    (fill (arc_segments 32) (thermal_gap 0.508) (thermal_bridge_width 0.508))
+    (polygon
+      (pts
+        (xy 193.775 186.175) (xy 193.775 180.375) (xy 227.045 180.375) (xy 227.045 85.975) (xy 201.625 85.975)
+        (xy 201.625 83.975) (xy 77.175 83.975) (xy 77.175 104.425) (xy 64.475 104.425) (xy 64.475 82.975)
+        (xy 232.125 82.975) (xy 232.125 181.375) (xy 205.525 181.375) (xy 205.525 186.175)
+      )
+    )

Commit message: templates
Changed lines of the file:
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@@
-(kicad_pcb (version 20171130) (host pcbnew 5.1.2-f72e74a~84~ubuntu16.04.1)
+(kicad_pcb (version 20171130) (host pcbnew 5.1.3-ffb9f22~84~ubuntu16.04.1)
   (general
     (thickness 1.6)
-    (drawings 51)
+    (drawings 52)
     (tracks 425)
     (zones 0)
@@
     (pad_to_mask_clearance 0.051)
     (solder_mask_min_width 0.25)
-    (aux_axis_origin 0 0)
-    (grid_origin 109.375 194.125)
+    (aux_axis_origin 109.625 194.125)
+    (grid_origin 109.625 194.125)
     (visible_elements FFFDFFFF)
     (pcbplotparams
@@
     )
   )
+  (target plus (at 109.625 194.125) (size 5) (width 0.05) (layer Edge.Cuts))
   (gr_line (start 232.1277 181.375) (end 205.525 181.375) (layer Edge.Cuts) (width 0.15))
   (gr_line (start 232.125 82.975) (end 232.1277 181.375) (layer Edge.Cuts) (width 0.15))
@@
     (polygon
       (pts
-        (xy 64.5 83) (xy 232.125 83) (xy 232.125 181.375) (xy 205.5 181.375) (xy 205.5 186.25)
-        (xy 193.75 186.25) (xy 193.75 188.625) (xy 109.375 188.625) (xy 109.375 183.25) (xy 105.875 183.25)
-        (xy 105.875 186.125) (xy 97.75 186.125) (xy 97.75 181.375) (xy 79.5 181.375) (xy 79.5 189.625)
+        (xy 64.5 83) (xy 232.125 83) (xy 232.125 181.375) (xy 205.5 181.375) (xy 205.5 186.125)
+        (xy 193.75 186.125) (xy 193.75 188.525) (xy 109.375 188.525) (xy 109.375 183.25) (xy 105.875 183.25)
+        (xy 105.875 186) (xy 97.75 186) (xy 97.75 181.375) (xy 79.5 181.375) (xy 79.5 189.625)
         (xy 64.5 189.625)
       )
@@
     (polygon
       (pts
-        (xy 64.5 83) (xy 232.125 83) (xy 232.125 181.375) (xy 205.5 181.375) (xy 205.5 186.25)
-        (xy 193.75 186.25) (xy 193.75 188.625) (xy 109.375 188.625) (xy 109.375 183.25) (xy 105.875 183.25)
-        (xy 105.875 186.125) (xy 97.75 186.125) (xy 97.75 181.375) (xy 79.5 181.375) (xy 79.5 189.625)
+        (xy 64.5 83) (xy 232.125 83) (xy 232.125 181.375) (xy 205.5 181.375) (xy 205.5 186.125)
+        (xy 193.75 186.125) (xy 193.75 188.525) (xy 109.375 188.525) (xy 109.375 183.25) (xy 105.875 183.25)
+        (xy 105.875 186) (xy 97.75 186) (xy 97.75 181.375) (xy 79.5 181.375) (xy 79.5 189.625)
         (xy 64.5 189.625)
       )
@@
     (polygon
       (pts
-        (xy 64.5 83) (xy 232.125 83) (xy 232.125 181.375) (xy 205.5 181.375) (xy 205.5 186.25)
-        (xy 193.75 186.25) (xy 193.75 188.625) (xy 109.375 188.625) (xy 109.375 183.25) (xy 105.875 183.25)
-        (xy 105.875 186.125) (xy 97.75 186.125) (xy 97.75 181.375) (xy 79.5 181.375) (xy 79.5 189.625)
+        (xy 64.5 83) (xy 232.125 83) (xy 232.125 181.375) (xy 205.5 181.375) (xy 205.5 186.125)
+        (xy 193.75 186.125) (xy 193.75 188.525) (xy 109.375 188.525) (xy 109.375 183.25) (xy 105.875 183.25)
+        (xy 105.875 186) (xy 97.75 186) (xy 97.75 181.375) (xy 79.5 181.375) (xy 79.5 189.625)
         (xy 64.5 189.625)
       )
@@
     (polygon
       (pts
-        (xy 64.5 83) (xy 232.125 83) (xy 232.125 181.375) (xy 205.5 181.375) (xy 205.5 186.25)
-        (xy 193.75 186.25) (xy 193.75 188.625) (xy 109.375 188.625) (xy 109.375 183.25) (xy 105.875 183.25)
-        (xy 105.875 186.125) (xy 97.75 186.125) (xy 97.75 181.375) (xy 79.5 181.375) (xy 79.5 189.625)
+        (xy 64.5 83) (xy 232.125 83) (xy 232.125 181.375) (xy 205.5 181.375) (xy 205.5 186.125)
+        (xy 193.75 186.125) (xy 193.75 188.525) (xy 109.375 188.525) (xy 109.375 183.25) (xy 105.875 183.25)
+        (xy 105.875 186) (xy 97.75 186) (xy 97.75 181.375) (xy 79.5 181.375) (xy 79.5 189.625)
         (xy 64.5 189.625)
       )

Commit message: KiCad 6 update
Connections:
- net /~PERST renamed /~{PERST}
- net /~PRSNT1 renamed /~{PRSNT1}
- net /~PRSNT2x1 renamed /~{PRSNT2x1}
- net /~PRSNT2x16 renamed /~{PRSNT2x16}
- net /~PRSNT2x4 renamed /~{PRSNT2x4}
- net /~PRSNT2x8 renamed /~{PRSNT2x8}
- net /~TRST renamed /~{TRST}
- net /~WAKE renamed /~{WAKE}
Other:
- net class Default removed
- net class Diff-100-PCIe removed
- net class JLC2313-100d-3.5 removed
- net class JLC2313-100d-4 removed
- net class JLC7628-100d-8 removed
